Commit message: updated limits to the manipulators except grippers

File: src/my_bot/description/manipulator.xacro (robot description, xacro)
@@ -29,5 +29,5 @@
         <child link="mnp_base_link"/>
         <axis xyz="0.0 0.0 1.0"/>
-        <limit lower="0" upper="0" effort="0.0" velocity="0.0"/>
+        <limit lower="-3.14" upper="3.14" effort="5" velocity="0.5"/>
     </joint>
 <!-- First Link -->
@@ -54,10 +54,10 @@
         <self_collide>1</self_collide>
     </gazebo>
-    <joint name="mnp_first_joint" type="continuous">
+    <joint name="mnp_first_joint" type="revolute">
         <origin xyz="0 0.0 0.15" rpy="0.0 0.0 0.0"/>
         <parent link="mnp_base_link"/>
         <child link="mnp_first_link"/>
         <axis xyz="0.0 1.0 0.0"/>
-        <limit lower="-1.57" upper="1.57" effort="5" velocity="0.5"/>
+        <limit lower="-1.5707" upper="1.5707" effort="5" velocity="0.5"/>
         <dynamics damping="0.7"/>
     </joint>
@@ -85,10 +85,10 @@
         <self_collide>1</self_collide>
     </gazebo>
-    <joint name="mnp_second_joint" type="continuous">
+    <joint name="mnp_second_joint" type="revolute">
         <origin xyz="0 0.05 1" rpy="0.0 0.0 0.0"/>
         <parent link="mnp_first_link"/>
         <child link="mnp_second_link"/>
         <axis xyz="0.0 1.0 0.0"/>
-        <limit lower="-1.57" upper="1.57" effort="5" velocity="0.5"/>
+        <limit lower="-1.5707" upper="1.5707" effort="5" velocity="0.5"/>
         <dynamics damping="0.7"/>
     </joint>
@@ -116,5 +116,5 @@
         <self_collide>1</self_collide>
     </gazebo>
-    <joint name="mnp_third_joint" type="continuous">
+    <joint name="mnp_third_joint" type="revolute">
         <origin xyz="0 0.05 .75" rpy="0.0 0.0 0.0"/>
         <parent link="mnp_second_link"/>

File: src/my_bot/description/ros2_control.xacro (robot description, xacro)
@@ -41,10 +41,11 @@
             <state_interface name="effort" />
         </joint>
-        <!-- <joint name="mnp_base_joint">
-            <command_interface name="position" />
+        <joint name="mnp_base_joint">
+            <command_interface name="position">
+                <param name="min">-3.14</param>
+                <param name="max">3.14</param>
+            </command_interface>
             <state_interface name="position" />
-            <state_interface name="velocity" />
-            <state_interface name="effort" />
-        </joint> -->
+        </joint>
         <joint name="mnp_first_joint">
             <command_interface name="position">
@@ -68,11 +69,5 @@
             <state_interface name="position" />
         </joint>
-        <!-- <joint name="mnp_ee_base_joint">
-            <command_interface name="position" />
-            <state_interface name="position" />
-            <state_interface name="velocity" />
-            <state_interface name="effort" />
-        </joint>
-        <joint name="mnp_left_gripper_joint">
+        <!-- <joint name="mnp_left_gripper_joint">
             <command_interface name="position" />
             <state_interface name="position" />
@@ -89,7 +84,6 @@
     <gazebo>
         <plugin name="gazebo_ros2_control" filename="libgazebo_ros2_control.so">
-            <self_collide>1</self_collide>
-            <!-- <robot_param>robot_description</robot_param>
-            <robot_param_node>robot_state_publisher</robot_param_node> -->
+            <robot_param>robot_description</robot_param>
+            <robot_param_node>robot_state_publisher</robot_param_node>
             <parameters>$(find my_bot)/config/mobile_manipulators.yaml</parameters>
         </plugin>
