Commit message: arm and sensor controller added

File: src/rover_sim/urdf/arm.xacro (robot description, xacro)
@@ -58,5 +58,6 @@
 		<limit lower="${-arm_01_limit}" upper="${arm_01_limit}" effort="10000.0" velocity="100.0"/>
         <axis xyz="0 0 1"/>
-        <joint_properties damping="0.0" friction="0.0"/>
+		<dynamics damping="0.5" />
+        <!-- <joint_properties damping="0.0" friction="0.0"/> -->
 	</joint>
     <!-- <transmission name="arm_01_trans">
@@ -126,5 +127,6 @@
 		<limit lower="${-arm_02_limit}" upper="${arm_02_limit}" effort="10000.0" velocity="100.0"/>
         <axis xyz="1 0 0"/>
-        <joint_properties damping="0.0" friction="0.0"/>
+		<dynamics damping="2" />
+        <!-- <joint_properties damping="2" friction="0.0"/> -->
 	</joint>
     <!-- <transmission name="arm_02_trans">
@@ -194,5 +196,6 @@
 		<limit lower="${-arm_03_limit}" upper="${arm_03_limit}" effort="10000.0" velocity="100.0"/>
         <axis xyz="1 0 0"/>
-        <joint_properties damping="0.0" friction="0.0"/>
+		<dynamics damping="0.5" />
+        <!-- <joint_properties damping="0.0" friction="0.0"/> -->
 	</joint>
     <!-- <transmission name="arm_03_trans">
@@ -262,5 +265,6 @@
 		<limit lower="${-arm_04_limit}" upper="${arm_04_limit}" effort="10000.0" velocity="100.0"/>
         <axis xyz="0 1 0"/>
-        <joint_properties damping="0.0" friction="0.0"/>
+		<dynamics damping="0.5" />
+        <!-- <joint_properties damping="0.0" friction="0.0"/> -->
 	</joint>
     <!-- <transmission name="arm_04_trans">
@@ -330,5 +334,6 @@
 		<limit effort="10000.0" velocity="100.0"/>
         <axis xyz="0 0 1"/>
-        <joint_properties damping="0.0" friction="0.0"/>
+		<dynamics damping="0.5" />
+        <!-- <joint_properties damping="0.0" friction="0.0"/> -->
 	</joint>
     <!-- <transmission name="arm_tools_trans">

File: src/rover_sim/urdf/left_wheel_group.xacro (robot description, xacro)
@@ -62,5 +62,5 @@
 		<joint_properties damping="${suspension_damping}" friction="${suspension_friction}"/>
 	</joint>
-	<transmission name="suspension_arm_F_L_trans">
+	<!-- <transmission name="suspension_arm_F_L_trans">
       <type>transmission_interface/SimpleTransmission</type>
       <joint name="suspension_arm_F_L_joint">
@@ -71,5 +71,5 @@
         <mechanicalReduction>1</mechanicalReduction>
       </actuator>
-    </transmission>
+    </transmission> -->
   	<link name='suspension_arm_B_L'>
 		<collision>
@@ -103,5 +103,5 @@
 		<joint_properties damping="${suspension_damping}" friction="${suspension_friction}"/>
 	</joint>
-	<transmission name="suspension_arm_B_L_trans">
+	<!-- <transmission name="suspension_arm_B_L_trans">
       <type>transmission_interface/SimpleTransmission</type>
       <joint name="suspension_arm_B_L_joint">
@@ -112,5 +112,5 @@
         <mechanicalReduction>1</mechanicalReduction>
       </actuator>
-    </transmission>
+    </transmission> -->
  	<link name='suspension_arm_B_L_to_B2_L'>
 		<inertial>
@@ -168,5 +168,5 @@
 		<joint_properties damping="${suspension_damping}" friction="${suspension_friction}"/>
 	</joint>
-	<transmission name="suspension_arm_B2_L_trans">
+	<!-- <transmission name="suspension_arm_B2_L_trans">
       <type>transmission_interface/SimpleTransmission</type>
       <joint name="suspension_arm_B2_L_joint">
@@ -177,5 +177,5 @@
         <mechanicalReduction>1</mechanicalReduction>
       </actuator>
-    </transmission>
+    </transmission> -->
 	<!-- FRONT WHEEL -->
 	<link name='suspension_arm_F_L_to_suspension_steer_F_L'>
@@ -233,5 +233,5 @@
         <axis xyz="0 0 1"/>
 	</joint>
-	<transmission name="suspension_steer_F_L_trans">
+	<!-- <transmission name="suspension_steer_F_L_trans">
       <type>transmission_interface/SimpleTransmission</type>
       <joint name="suspension_steer_F_L_joint">
@@ -242,5 +242,5 @@
         <mechanicalReduction>1</mechanicalReduction>
       </actuator>
-    </transmission>
+    </transmission> -->
 	<link name='suspension_steer_F_L_to_front_wheel_L'>
 		<inertial>
@@ -358,5 +358,5 @@
         <axis xyz="0 0 1"/>
 	</joint>
-	<transmission name="suspension_steer_B_L_trans">
+	<!-- <transmission name="suspension_steer_B_L_trans">
       <type>transmission_interface/SimpleTransmission</type>
       <joint name="suspension_steer_B_L_joint">
@@ -367,5 +367,5 @@
         <mechanicalReduction>1</mechanicalReduction>
       </actuator>
-    </transmission>
+    </transmission> -->
   	<link name='suspension_steer_B_L_to_back_wheel_L'>
 		<inertial>

File: src/rover_sim/urdf/right_wheel_group.xacro (robot description, xacro)
@@ -67,5 +67,5 @@
 		<joint_properties damping="${suspension_damping}" friction="${suspension_friction}"/>
 	</joint>
-  	<transmission name="suspension_arm_F_R_trans">
+  	<!-- <transmission name="suspension_arm_F_R_trans">
       <type>transmission_interface/SimpleTransmission</type>
       <joint name="suspension_arm_F_R_joint">
@@ -76,5 +76,5 @@
         <mechanicalReduction>1</mechanicalReduction>
       </actuator>
-    </transmission>
+    </transmission> -->
   	<link name='suspension_arm_B_R'>
 		<collision>
@@ -111,5 +111,5 @@
 		<joint_properties damping="${suspension_damping}" friction="${suspension_friction}"/>
 	</joint>
-  	<transmission name="suspension_arm_B_R_trans">
+  	<!-- <transmission name="suspension_arm_B_R_trans">
       <type>transmission_interface/SimpleTransmission</type>
       <joint name="suspension_arm_B_R_joint">
@@ -120,5 +120,5 @@
         <mechanicalReduction>1</mechanicalReduction>
       </actuator>
-    </transmission>
+    </transmission> -->
   	<link name='suspension_arm_B_R_to_B2_R'>
 		<inertial>
@@ -179,5 +179,5 @@
 		<joint_properties damping="${suspension_damping}" friction="${suspension_friction}"/>
 	</joint>
-  	<transmission name="suspension_arm_B2_R_trans">
+  	<!-- <transmission name="suspension_arm_B2_R_trans">
       <type>transmission_interface/SimpleTransmission</type>
       <joint name="suspension_arm_B2_R_joint">
@@ -188,5 +188,5 @@
         <mechanicalReduction>1</mechanicalReduction>
       </actuator>
-    </transmission>
+    </transmission> -->
 	<!-- FRONT WHEEL RIGHT -->
 	<link name='suspension_arm_F_R_to_suspension_steer_F_R'>
@@ -247,5 +247,5 @@
         <axis xyz="0 0 1"/>
 	</joint>
-	<transmission name="suspension_steer_F_R_trans">
+	<!-- <transmission name="suspension_steer_F_R_trans">
       <type>transmission_interface/SimpleTransmission</type>
       <joint name="suspension_steer_F_R_joint">
@@ -256,5 +256,5 @@
         <mechanicalReduction>1</mechanicalReduction>
       </actuator>
-    </transmission>
+    </transmission> -->
 	<link name='suspension_steer_F_R_to_front_wheel_R'>
 		<inertial>
@@ -372,5 +372,5 @@
         <axis xyz="0 0 1"/>
 	</joint>
-  	<transmission name="suspension_steer_B_R_trans">
+  	<!-- <transmission name="suspension_steer_B_R_trans">
       <type>transmission_interface/SimpleTransmission</type>
       <joint name="suspension_steer_B_R_joint">
@@ -381,5 +381,5 @@
         <mechanicalReduction>1</mechanicalReduction>
       </actuator>
-    </transmission>
+    </transmission> -->
 	<link name='suspension_steer_B_R_to_back_wheel_R'>
 		<inertial>

File: src/rover_sim/urdf/rover.gazebo.xacro (robot description, xacro)
@@ -1,21 +1,169 @@
 <?xml version="1.0"?>
-<robot xmlns:xacro="http://www.ros.org/wiki/xacro">
-  <!-- ros_control plugin -->
-  <gazebo>
-    <plugin name="gazebo_ros_control" filename="libgazebo_ros_control.so">
-      <robotNamespace>/rover</robotNamespace>
-      <robotParam>/robot_description</robotParam>
-      <robotSimType>gazebo_ros_control/DefaultRobotHWSim</robotSimType>
-    </plugin>
-  </gazebo>
+<robot xmlns:xacro="http://www.ros.org/wiki/xacro" >
+    <ros2_control name="GazeboSystem" type="system">
+        <hardware>
+            <plugin>gazebo_ros2_control/GazeboSystem</plugin>
+        </hardware>
+        <joint name="mast_p_joint">
+            <command_interface name="position">
+                <param name="min">0</param>
+                <param name="max">1.57</param>
+            </command_interface>
+            <state_interface name="position" />
+        </joint>
+        <joint name="mast_02_joint">
+            <command_interface name="position">
+                <param name="min">-3.14</param>
+                <param name="max">3.14</param>
+            </command_interface>
+            <state_interface name="position" />
+        </joint>
+        <joint name="mast_cameras_joint">
+            <command_interface name="position">
+                <param name="min">-1.57</param>
+                <param name="max">1.57</param>
+            </command_interface>
+            <state_interface name="position" />
+        </joint>
+        <!--  -->
+        <joint name="arm_01_joint">
+            <command_interface name="position">
+                <param name="min">-1.57</param>
+                <param name="max">1.57</param>
+            </command_interface>
+            <state_interface name="position" />
+        </joint>
+        <joint name="arm_02_joint">
+            <command_interface name="position">
+                <param name="min">-1.57</param>
+                <param name="max">1.57</param>
+            </command_interface>
+            <state_interface name="position" />
+        </joint>
+        <joint name="arm_03_joint">
+            <command_interface name="position">
+                <param name="min">-1.57</param>
+                <param name="max">1.57</param>
+            </command_interface>
+            <state_interface name="position" />
+        </joint>
+        <joint name="arm_04_joint">
+            <command_interface name="position">
+                <param name="min">-1.57</param>
+                <param name="max">1.57</param>
+            </command_interface>
+            <state_interface name="position" />
+        </joint>
+        <joint name="arm_tools_joint">
+            <command_interface name="position">
+                <param name="min">-3.14</param>
+                <param name="max">3.14</param>
+            </command_interface>
+            <state_interface name="position" />
+        </joint>
+    </ros2_control>
+    <gazebo>
+        <plugin name="gazebo_ros2_control" filename="libgazebo_ros2_control.so">
+            <robot_param>robot_description</robot_param>
+            <robot_param_node>robot_state_publisher</robot_param_node>
+            <parameters>$(find rover_sim)/config/rover_controller.yaml</parameters>
+        </plugin>
+    </gazebo>
+  <!-- Friction values -->
+  <!-- Chassis -->
+  <gazebo reference="chassis">
+    <mu1>0.3</mu1>
+    <mu2>0.3</mu2>
+  </gazebo>
+  <!-- Wheel Train -->
+  <gazebo reference="left_axis">
+    <mu1>0.3</mu1>
+    <mu2>0.3</mu2>
+  </gazebo>
+  <gazebo reference="suspension_arm_F_L">
+    <mu1>0.3</mu1>
+    <mu2>0.3</mu2>
+  </gazebo>
+  <gazebo reference="right_axis">
+    <mu1>0.3</mu1>
+    <mu2>0.3</mu2>
+  </gazebo>
+  <gazebo reference="suspension_arm_F_R">
+    <mu1>0.3</mu1>
+    <mu2>0.3</mu2>
+  </gazebo>
+  <gazebo reference="suspension_arm_B_L">
+    <mu1>0.3</mu1>
+    <mu2>0.3</mu2>
+  </gazebo>
+  <gazebo reference="suspension_arm_B_R">
+    <mu1>0.3</mu1>
+    <mu2>0.3</mu2>
+  </gazebo>
+  <gazebo reference="suspension_arm_B_L_to_B2_L">
+    <mu1>0.3</mu1>
+    <mu2>0.3</mu2>
+    <material>Gazebo/Black</material>
+  </gazebo>
+  <gazebo reference="suspension_arm_B_R_to_B2_R">
+    <mu1>0.3</mu1>
+    <mu2>0.3</mu2>
+    <material>Gazebo/Black</material>
+  </gazebo>
+  <gazebo reference="suspension_arm_B2_L">
+    <mu1>0.3</mu1>
+    <mu2>0.3</mu2>
+  </gazebo>
+  <gazebo reference="suspension_arm_B2_R">
+    <mu1>0.3</mu1>
+    <mu2>0.3</mu2>
+  </gazebo>
+  <gazebo reference="suspension_arm_F_L_to_suspension_steer_F_L">
+    <mu1>0.3</mu1>
+    <mu2>0.3</mu2>
+  </gazebo>
+  <gazebo reference="suspension_arm_F_R_to_suspension_steer_F_R">
+    <mu1>0.3</mu1>
+    <mu2>0.3</mu2>
+  </gazebo>
+  <gazebo reference="suspension_steer_F_L">
+    <mu1>0.3</mu1>
+    <mu2>0.3</mu2>
+  </gazebo>
+  <gazebo reference="suspension_steer_F_R">
+    <mu1>0.3</mu1>
+    <mu2>0.3</mu2>
+  </gazebo>
+  <gazebo reference="suspension_arm_B2_L_to_suspension_steer_B_L">
+    <mu1>0.3</mu1>
+    <mu2>0.3</mu2>
+  </gazebo>
+  <gazebo reference="suspension_arm_B2_R_to_suspension_steer_B_R">
+    <mu1>0.3</mu1>
+    <mu2>0.3</mu2>
+  </gazebo>
+  <gazebo reference="suspension_steer_B_L">
+    <mu1>0.3</mu1>
+    <mu2>0.3</mu2>
+  </gazebo>
+  <gazebo reference="suspension_steer_B_R">
+    <mu1>0.3</mu1>
+    <mu2>0.3</mu2>
+  </gazebo>
+  <!-- Arm -->
+  <gazebo reference="arm_01">
+    <mu1>0.3</mu1>
+    <mu2>0.3</mu2>
+  </gazebo>
+  </robot>
   <!--
     The plugin broadcasts a body's pose and rates through ROS nav_msgs::Odometry message.
     The plugin broadcasts pose and rate of a body named "chassis" over ROS topic name "curiosity_mars_rover/odom".
   -->
-  <gazebo>
+  <!-- <gazebo>
     <plugin name="ground_truth"
             filename="libgazebo_ros_p3d.so">
       <frameName>world</frameName>
-        <!-- here world is what? can be an issue too -->
+        here world is what? can be an issue too
       <bodyName>chassis</bodyName>
       <topicName>/rover/odom</topicName>
@@ -58,90 +206,3 @@
       </plugin>
     </sensor>
-  </gazebo>
-<!-- Friction values -->
-  <!-- Chassis -->
-  <gazebo reference="chassis">
-    <mu1>0.3</mu1>
-    <mu2>0.3</mu2>
-  </gazebo>
-  <!-- Wheel Train -->
-  <gazebo reference="left_axis">
-    <mu1>0.3</mu1>
-    <mu2>0.3</mu2>
-  </gazebo>
-  <gazebo reference="suspension_arm_F_L">
-    <mu1>0.3</mu1>
-    <mu2>0.3</mu2>
-  </gazebo>
-  <gazebo reference="right_axis">
-    <mu1>0.3</mu1>
-    <mu2>0.3</mu2>
-  </gazebo>
-  <gazebo reference="suspension_arm_F_R">
-    <mu1>0.3</mu1>
-    <mu2>0.3</mu2>
-  </gazebo>
-  <gazebo reference="suspension_arm_B_L">
-    <mu1>0.3</mu1>
-    <mu2>0.3</mu2>
-  </gazebo>
-  <gazebo reference="suspension_arm_B_R">
-    <mu1>0.3</mu1>
-    <mu2>0.3</mu2>
-  </gazebo>
-  <gazebo reference="suspension_arm_B_L_to_B2_L">
-    <mu1>0.3</mu1>
-    <mu2>0.3</mu2>
-    <material>Gazebo/Black</material>
-  </gazebo>
-  <gazebo reference="suspension_arm_B_R_to_B2_R">
-    <mu1>0.3</mu1>
-    <mu2>0.3</mu2>
-    <material>Gazebo/Black</material>
-  </gazebo>
-  <gazebo reference="suspension_arm_B2_L">
-    <mu1>0.3</mu1>
-    <mu2>0.3</mu2>
-  </gazebo>
-  <gazebo reference="suspension_arm_B2_R">
-    <mu1>0.3</mu1>
-    <mu2>0.3</mu2>
-  </gazebo>
-  <gazebo reference="suspension_arm_F_L_to_suspension_steer_F_L">
-    <mu1>0.3</mu1>
-    <mu2>0.3</mu2>
-  </gazebo>
-  <gazebo reference="suspension_arm_F_R_to_suspension_steer_F_R">
-    <mu1>0.3</mu1>
-    <mu2>0.3</mu2>
-  </gazebo>
-  <gazebo reference="suspension_steer_F_L">
-    <mu1>0.3</mu1>
-    <mu2>0.3</mu2>
-  </gazebo>
-  <gazebo reference="suspension_steer_F_R">
-    <mu1>0.3</mu1>
-    <mu2>0.3</mu2>
-  </gazebo>
-  <gazebo reference="suspension_arm_B2_L_to_suspension_steer_B_L">
-    <mu1>0.3</mu1>
-    <mu2>0.3</mu2>
-  </gazebo>
-  <gazebo reference="suspension_arm_B2_R_to_suspension_steer_B_R">
-    <mu1>0.3</mu1>
-    <mu2>0.3</mu2>
-  </gazebo>
-  <gazebo reference="suspension_steer_B_L">
-    <mu1>0.3</mu1>
-    <mu2>0.3</mu2>
-  </gazebo>
-  <gazebo reference="suspension_steer_B_R">
-    <mu1>0.3</mu1>
-    <mu2>0.3</mu2>
-  </gazebo>
-  <!-- Arm -->
-  <gazebo reference="arm_01">
-    <mu1>0.3</mu1>
-    <mu2>0.3</mu2>
-  </gazebo>
-</robot>
+  </gazebo> -->

File: src/rover_sim/urdf/rover.urdf.xacro (robot description, xacro)
@@ -3,5 +3,5 @@
 	<xacro:include filename="$(find rover_sim)/urdf/macros.xacro"/>
 	<xacro:include filename="$(find rover_sim)/urdf/properties.xacro"/>
-    <!-- <xacro:include filename="$(find rover_sim)/urdf/rover.gazebo.xacro"/> -->
+    <xacro:include filename="$(find rover_sim)/urdf/rover.gazebo.xacro"/>
     <xacro:include filename="$(find rover_sim)/urdf/chassis.xacro"/>
     <xacro:include filename="$(find rover_sim)/urdf/wheel.xacro"/>

File: src/rover_sim/urdf/sensors.xacro (robot description, xacro)
@@ -59,5 +59,6 @@
         <!-- <limit lower="0" upper="0.05" effort="10000.0" velocity="100.0"/> -->
         <axis xyz="0 1 0"/>
-        <joint_properties damping="0" friction="0"/>
+		<dynamics damping="0.5" />
+        <!-- <joint_properties damping="0" friction="0"/> -->
 	</joint>
     <!-- <transmission name="mast_p_trans">
@@ -127,5 +128,6 @@
 		<limit effort="10000.0" velocity="100.0"/>
         <axis xyz="0 0 1"/>
-        <joint_properties damping="0.0" friction="0.0"/>
+		<dynamics damping="0.5" />
+        <!-- <joint_properties damping="0.0" friction="0.0"/> -->
 	</joint>
     <!-- <transmission name="mast_02_trans">
@@ -195,5 +197,6 @@
 		<limit lower="${-mast_cameras_limit}" upper="${mast_cameras_limit}" effort="10000.0" velocity="100.0"/>
         <axis xyz="1 0 0"/>
-        <joint_properties damping="0.0" friction="0.0"/>
+		<dynamics damping="0.5" />
+        <!-- <joint_properties damping="0.0" friction="0.0"/> -->
 	</joint>
     <!-- <transmission name="mast_02_trans">

File: src/rover_sim/urdf/wheel.xacro (robot description, xacro)
@@ -43,5 +43,5 @@
         <joint_properties damping="0.0" friction="0.0"/>
 	</joint>
-    <transmission name="${wheel_name}_trans">
+    <!-- <transmission name="${wheel_name}_trans">
       <type>transmission_interface/SimpleTransmission</type>
       <joint name="${wheel_name}_joint">
@@ -52,5 +52,5 @@
         <mechanicalReduction>1</mechanicalReduction>
       </actuator>
-    </transmission>
+    </transmission> -->
   </xacro:macro>
 </robot>
