Commit message: skid controller added

File: src/rover_sim/urdf/rover.gazebo.xacro (robot description, xacro)
@@ -5,4 +5,58 @@
             <plugin>gazebo_ros2_control/GazeboSystem</plugin>
         </hardware>
+        <joint name="front_wheel_L_joint">
+            <command_interface name="velocity">
+                <param name="min">-50</param>
+                <param name="max">50</param>
+            </command_interface>
+            <state_interface name="position" />
+            <state_interface name="velocity" />
+            <state_interface name="effort" />
+        </joint>
+        <joint name="middle_wheel_L_joint">
+            <command_interface name="velocity">
+                <param name="min">-50</param>
+                <param name="max">50</param>
+            </command_interface>
+            <state_interface name="position" />
+            <state_interface name="velocity" />
+            <state_interface name="effort" />
+        </joint>
+        <joint name="back_wheel_L_joint">
+            <command_interface name="velocity">
+                <param name="min">-50</param>
+                <param name="max">50</param>
+            </command_interface>
+            <state_interface name="position" />
+            <state_interface name="velocity" />
+            <state_interface name="effort" />
+        </joint>
+        <joint name="front_wheel_R_joint">
+            <command_interface name="velocity">
+                <param name="min">-50</param>
+                <param name="max">50</param>
+            </command_interface>
+            <state_interface name="position" />
+            <state_interface name="velocity" />
+            <state_interface name="effort" />
+        </joint>
+        <joint name="middle_wheel_R_joint">
+            <command_interface name="velocity">
+                <param name="min">-50</param>
+                <param name="max">50</param>
+            </command_interface>
+            <state_interface name="position" />
+            <state_interface name="velocity" />
+            <state_interface name="effort" />
+        </joint>
+        <joint name="back_wheel_R_joint">
+            <command_interface name="velocity">
+                <param name="min">-50</param>
+                <param name="max">50</param>
+            </command_interface>
+            <state_interface name="position" />
+            <state_interface name="velocity" />
+            <state_interface name="effort" />
+        </joint>
         <joint name="mast_p_joint">
             <command_interface name="position">
